Commit message: add dualarm_reach.py

File: assets/dualarm/bifranka_robot.urdf (robot description, URDF)
Before this commit: robot bifranka_robot, 24 links, 23 joints
Links:
- link base_link: geometry collision mesh filename=meshes/collision/base_mount.stl scale=0.001 0.001 0.001; visual mesh filename=meshes/visual/base_mount.dae
- link lewis_fr3_link0: geometry collision mesh filename=meshes/collision/link0.stl; visual mesh filename=meshes/visual/link0.dae
- link lewis_fr3_link1: geometry collision mesh filename=meshes/collision/link1.stl; visual mesh filename=meshes/visual/link1.dae
- link lewis_fr3_link2: geometry collision mesh filename=meshes/collision/link2.stl; visual mesh filename=meshes/visual/link2.dae
- link lewis_fr3_link3: geometry collision mesh filename=meshes/collision/link3.stl; visual mesh filename=meshes/visual/link3.dae
- link lewis_fr3_link4: geometry collision mesh filename=meshes/collision/link4.stl; visual mesh filename=meshes/visual/link4.dae
- link lewis_fr3_link5: geometry collision mesh filename=meshes/collision/link5.stl; visual mesh filename=meshes/visual/link5.dae
- link lewis_fr3_link6: geometry collision mesh filename=meshes/collision/link6.stl; visual mesh filename=meshes/visual/link6.dae
- link lewis_fr3_link7: geometry collision mesh filename=meshes/collision/link7.stl; visual mesh filename=meshes/visual/link7.dae
- link richard_fr3_link0: geometry collision mesh filename=meshes/collision/link0.stl; visual mesh filename=meshes/visual/link0.dae
- link richard_fr3_link1: geometry collision mesh filename=meshes/collision/link1.stl; visual mesh filename=meshes/visual/link1.dae
- link richard_fr3_link2: geometry collision mesh filename=meshes/collision/link2.stl; visual mesh filename=meshes/visual/link2.dae
- link richard_fr3_link3: geometry collision mesh filename=meshes/collision/link3.stl; visual mesh filename=meshes/visual/link3.dae
- link richard_fr3_link4: geometry collision mesh filename=meshes/collision/link4.stl; visual mesh filename=meshes/visual/link4.dae
- link richard_fr3_link5: geometry collision mesh filename=meshes/collision/link5.stl; visual mesh filename=meshes/visual/link5.dae
- link richard_fr3_link6: geometry collision mesh filename=meshes/collision/link6.stl; visual mesh filename=meshes/visual/link6.dae
- link richard_fr3_link7: geometry collision mesh filename=meshes/collision/link7.stl; visual mesh filename=meshes/visual/link7.dae

Commit message: fix dualarm model in the isaacgym

File: assets/dualarm/bifranka_robot.urdf (robot description, URDF)
Before this commit: robot bifranka_robot, 24 links, 23 joints
Links:
- link base_link: geometry collision mesh filename=meshes/collision/base_mount.stl scale=0.001 0.001 0.001; visual mesh filename=meshes/visual/base_mount.obj
